Commit message: has only one box as end-eff

File: omnigrasper_no_hook.urdf (robot description, URDF)
Before this commit: robot omnigrasper, 12 links, 11 joints
Links:
- added link arm_link, mass 0.06; collision box size=0.02 0.13 0.025; visual box size=0.02 0.13 0.025
Joints:
- added joint arm_5_end: type fixed, parent arm_5, child arm_link, origin xyz=0 0.039 -0.006
